Commit message: Added camera tool to URDF and corrected A6 transformation

File: rx60b_description/robots/rx60b_description.URDF (robot description, URDF)
Before this commit: robot RX60B-HB_5, 7 links, 6 joints
Links:
- added link bumblebee_cam1
- added link bumblebee_cam2
- added link cameratool; collision mesh filename=package://rx60b_description/meshes/tool_boundingbox.stl; visual mesh filename=package://rx60b_description/meshes/tool_visual.stl
Joints:
- added joint bumblebee_cam1_joint: type fixed, parent cameratool, child bumblebee_cam1, origin xyz=0.06 -0.016 0.106114 rpy=0 0 0, axis 1 0 0
- added joint bumblebee_cam2_joint: type fixed, parent cameratool, child bumblebee_cam2, origin xyz=-0.06 -0.016 0.106114 rpy=0 0 0, axis 1 0 0
- added joint toolmount: type fixed, parent tool_flange, child cameratool, origin xyz=0 0 0.0095 rpy=0 0 0, axis 1 0 0
- joint a5: origin xyz=0 0 0.2 rpy=3.14159265359 1.57079632679 0 -> xyz=0 0 0.2 rpy=0 1.57079632679 0

Commit message: Camera transforms in URDF file updated

File: rx60b_description/robots/rx60b_description.URDF (robot description, URDF)
Before this commit: robot RX60B-HB_5, 10 links, 9 joints
Links:
- added link asus_depthcam
- added link asus_projector
- added link asus_rgbcam
- added link camera_link
Joints:
- added joint asus_depthcam_joint: type fixed, parent cameratool, child asus_depthcam, origin xyz=-0.046 0.052 0.056 rpy=1.57079632679 0 3.14159265359, axis 1 0 0
- added joint asus_projector_joint: type fixed, parent cameratool, child asus_projector, origin xyz=0.0274 0.052 0.056 rpy=1.57079632679 0 3.14159265359, axis 1 0 0
- added joint asus_rgbcam_joint: type fixed, parent cameratool, child asus_rgbcam, origin xyz=-0.0196 0.052 0.056 rpy=1.57079632679 0 3.14159265359, axis 1 0 0
- added joint camera_link_joint: type fixed, parent cameratool, child camera_link, origin xyz=0.0 0.052 0.056 rpy=0 0 0, axis 1 0 0
- joint bumblebee_cam1_joint: origin xyz=0.06 -0.016 0.106114 rpy=0 0 0 -> xyz=-0.06 0.0 0.106114 rpy=-1.57079632679 0 0
- joint bumblebee_cam2_joint: origin xyz=-0.06 -0.016 0.106114 rpy=0 0 0 -> xyz=0.06 0.0 0.106114 rpy=-1.57079632679 0 0
- joint toolmount: origin xyz=0 0 0.0095 rpy=0 0 0 -> xyz=0 0 0.0095 rpy=0 0 -0.785398163

Commit message: Updated joint limits on A3 and A5

File: rx60b_description/robots/rx60b_description.URDF (robot description, URDF)
Before this commit: robot RX60B-HB_5, 14 links, 13 joints
Joints:
- joint a3: limit lower=-3.14159265359 upper=3.14159265359 effort=0 velocity=0.1 -> lower=-2.2 upper=2.2 effort=0 velocity=0.1
- joint a5: limit lower=-4.71238898 upper=4.71238898 effort=0 velocity=0.1 -> lower=-2 upper=2 effort=0 velocity=0.1

Commit message: Transformations about a6 corrected

File: rx60b_description/robots/rx60b_description.URDF (robot description, URDF)
Before this commit: robot RX60B-HB_5, 14 links, 13 joints
Joints:
- joint a5: origin xyz=0 0 0.2 rpy=0 1.57079632679 0 -> xyz=0 0 0.2 rpy=3.14159265359 1.57079632679 0
- joint a6: origin xyz=-0.07 0 0 rpy=0 -1.57079632679 0 -> xyz=-0.07 0 0 rpy=0 1.57079632679 3.14159265359
- joint camera_link_joint: origin xyz=0.0 0.052 0.056 rpy=0 0 0 -> xyz=0.0 0.052 0.056 rpy=0 0 1.57079632679

Commit message: Controller and moveit updated to support higher joint velocities

File: rx60b_description/robots/rx60b_description.URDF (robot description, URDF)
Before this commit: robot RX60B-HB_5, 14 links, 13 joints
Joints:
- joint a1: limit lower=-3.14159265359 upper=3.14159265359 effort=0 velocity=0.1 -> lower=-3.14159265359 upper=3.14159265359 effort=0 velocity=0.2
- joint a2: limit lower=-2.0943951 upper=2.0943951 effort=0 velocity=0.1 -> lower=-2.0943951 upper=2.0943951 effort=0 velocity=0.2
- joint a3: limit lower=-2.2 upper=2.2 effort=0 velocity=0.1 -> lower=-2.2 upper=2.2 effort=0 velocity=0.2
- joint a4: limit lower=-2.3387412 upper=2.3387412 effort=0 velocity=0.1 -> lower=-2.3387412 upper=2.3387412 effort=0 velocity=0.2
- joint a5: limit lower=-2 upper=2 effort=0 velocity=0.1 -> lower=-2 upper=2 effort=0 velocity=0.2
- joint a6: limit lower=-2.0943951 upper=2.0943951 effort=0 velocity=0.1 -> lower=-2.0943951 upper=2.0943951 effort=0 velocity=0.2

Commit message: RX60B robot model updated cleaned and draft power connector added to collision mode

File: rx60b_description/robots/rx60b_description.URDF (robot description, URDF)
Before this commit: robot RX60B-HB_5, 14 links, 13 joints
Links:
- added link powerconnector; collision mesh filename=package://rx60b_description/meshes/powerconnector.stl
- link arm: geometry collision mesh filename=package://rx60b_description/meshes/arm.stl; visual mesh filename=package://rx60b_description/meshes/arm.stl
- link base_link: geometry collision mesh filename=package://rx60b_description/meshes/base_link.stl; visual mesh filename=package://rx60b_description/meshes/base_link.stl
- link elbow: geometry collision mesh filename=package://rx60b_description/meshes/elbow.stl; visual mesh filename=package://rx60b_description/meshes/elbow.stl
- link forearm: geometry collision mesh filename=package://rx60b_description/meshes/forearm.stl; visual mesh filename=package://rx60b_description/meshes/forearm.stl
- link shoulder: geometry collision mesh filename=package://rx60b_description/meshes/shoulder.stl; visual mesh filename=package://rx60b_description/meshes/shoulder.stl
- link wrist: geometry collision mesh filename=package://rx60b_description/meshes/wrist.stl; visual mesh filename=package://rx60b_description/meshes/wrist.stl
Joints:
- added joint powerconnector_joint: type fixed, parent base_link, child powerconnector, origin xyz=-0.15 0 0.09 rpy=1.57079632679 1.57079632679 0, axis 1 0 0

Commit message: Updated for first beta

File: rx60b_description/robots/rx60b_description.URDF (robot description, URDF)
Before this commit: robot RX60B-HB_5, 15 links, 14 joints
Links:
- added link collision_object; collision cylinder length=0.15 radius=0.08
Joints:
- added joint collision_object_joint: type fixed, parent base_link, child collision_object, origin xyz=0.0 0.0 0.75 rpy=0 0 0, axis 1 0 0

Commit message: Workcell collision objects added to robot description

File: rx60b_description/robots/rx60b_description.URDF (robot description, URDF)
Before this commit: robot RX60B-HB_5, 16 links, 15 joints
Links:
- added link collision_fence; collision box size=2 0.1 2
- added link collision_pole; collision box size=0.3 0.3 2
- added link collision_radiator; collision box size=0.3 2 0.52
- added link collision_table; collision box size=1.5 1.5 0.1
- added link collision_wall; collision box size=0.01 2 2
Joints:
- added joint collision_fence_joint: type fixed, parent base_link, child collision_fence, origin xyz=0.0 -0.79 0 rpy=0 0 0, axis 1 0 0
- added joint collision_pole_joint: type fixed, parent base_link, child collision_pole, origin xyz=-0.65 -0.7 0 rpy=0 0 0, axis 1 0 0
- added joint collision_radiator_joint: type fixed, parent base_link, child collision_radiator, origin xyz=-0.65 0.0 0.0 rpy=0 0 0, axis 1 0 0
- added joint collision_table_joint: type fixed, parent base_link, child collision_table, origin xyz=0.0 0.0 -0.025 rpy=0 0 0, axis 1 0 0
- added joint collision_wall_joint: type fixed, parent base_link, child collision_wall, origin xyz=-0.65 0 0 rpy=0 0 0, axis 1 0 0

Commit message: Changes made for the last testing - collision object removed due to the hand-eye calibration

File: rx60b_description/robots/rx60b_description.URDF (robot description, URDF)
Before this commit: robot RX60B-HB_5, 21 links, 20 joints
Links:
- removed link collision_object
Joints:
- removed joint collision_object_joint

Commit message: Files used for chessboard test added

File: rx60b_description/robots/rx60b_description.URDF (robot description, URDF)
Before this commit: robot RX60B-HB_5, 20 links, 19 joints
Links:
- added link camera_link_base
Joints:
- added joint camera_link_calibration_joint: type fixed, parent camera_link_base, child camera_link, origin xyz=-0.000720925758209 -0.0152323263351 0.0157927251061 rpy=-0.0168287298647 0.000769727110753 -0.096552431091, axis 1 0 0
- joint camera_link_joint: child camera_link -> camera_link_base
